File: RP2040_8key.kicad_pcb (KiCad board)
At the start: 2 copper layers, 110 x 38.3 mm, 55 parts, among them J1 USB_C_Receptacle, J2 AudioJack4, J3 Conn_01x03_Male, J4 Conn_01x03_Male, J5 TP1, J6 TP2, J7 TP3, SW1 SW_Push, SW10 RESET, SW2 SW_Push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

Commit message: Update 2023Version
Parts:
- C1, C2: footprint Capacitor_SMD:C_0402_1005Metric -> Capacitor_SMD:C_1206_3216Metric
- moved C1 1.90 mm to (191.6, 116.4), turned to -90 degrees
- moved C2 1.90 mm to (189.1, 116.4), turned to -90 degrees
Connections:
- net Net-(D4-Pad2) renamed rotary
Routing:
- net GND: track 29.9 -> 27.5 mm, vias 20 -> 19
- net +3V3: track 104.0 -> 102.3 mm, vias 4 -> 3
- net rotary: track 11.5 -> 13.1 mm
- net col3: track 55.2 -> 54.2 mm
- net row0: track 73.0 -> 73.9 mm
- net +5V: track 29.0 -> 29.8 mm
