File: RP2040_8key.kicad_sch (KiCad schematic)
At the start: 55 parts, among them J1 USB_C_Receptacle, J2 AudioJack4, J3 Conn_01x03_Male, J4 Conn_01x03_Male, J5 TP1, J6 TP2, J7 TP3, SW1 SW_Push, SW10 RESET, SW2 SW_Push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

Commit message: Update 2023Version
Parts:
- C1, C2: footprint Capacitor_SMD:C_0402_1005Metric -> Capacitor_SMD:C_1206_3216Metric
Connections:
- net rotary: now reaches D4.2 (A), SW4.2
Other:
- moved on the sheet: D1, D2, D3, D4, D5, D6, D7, D8, SW1, SW2, SW3, SW4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
